File: Sensor Boards/sensors.kicad_sch (KiCad schematic)
At the start: 11 parts, among them J1 Conn_Sensors, U1 LSM6DSM, U2 ADC081C021CIMM

Commit message: add MPNs for sensor board components - rts4
Parts:
- C1: MPN (none) -> 0402W106M6R3HI
- C2, C3, C4: MPN (none) -> 0402B104K160HI
- J1: MPN (none) -> B4B-XH-A
- R1, R2: MPN (none) -> RC0402JR-074K7L
- R3: MPN (none) -> RC0402JR-07100KL
- TH1: MPN (none) -> NCU15XH103F6SRC
- U1: MPN (none) -> LSM6DSVTR
- U2: MPN (none) -> ADC081C021CIMM/NOPB
Changed lines of the file:
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@@
+			)
+		)
+		(property "MPN" "LSM6DSVTR"
+			(at 115.57 87.63 0)
+			(effects
+				(font
+					(size 1.27 1.27)
+				)
+				(hide yes)
 			)
 		)
@@
 			)
 		)
+		(property "MPN" "0402W106M6R3HI"
+			(at 180.34 76.2 0)
+			(effects
+				(font
+					(size 1.27 1.27)
+				)
+				(hide yes)
+			)
+		)
 		(pin "2"
 		)
@@
 			)
 		)
+		(property "MPN" "B4B-XH-A"
+			(at 180.34 87.63 0)
+			(effects
+				(font
+					(size 1.27 1.27)
+				)
+				(hide yes)
+			)
+		)
 		(pin "3"
 		)
@@
 			)
 		)
+		(property "MPN" "0402B104K160HI"
+			(at 133.35 68.58 0)
+			(effects
+				(font
+					(size 1.27 1.27)
+				)
+				(hide yes)
+			)
+		)
 		(pin "2"
 		)
@@
 			)
 		)
+		(property "MPN" "RC0402JR-074K7L"
+			(at 163.83 93.98 0)
+			(effects
+				(font
+					(size 1.27 1.27)
+				)
+				(hide yes)
+			)
+		)
 		(pin "1"
 		)
@@
 			)
 		)
+		(property "MPN" "RC0402JR-074K7L"
+			(at 163.83 81.28 0)
+			(effects
+				(font
+					(size 1.27 1.27)
+				)
+				(hide yes)
+			)
+		)
 		(pin "1"
 		)
@@
 		)
 		(property "Description" "Unpolarized capacitor"
+			(at 146.05 116.84 0)
+			(effects
+				(font
+					(size 1.27 1.27)
+				)
+				(hide yes)
+			)
+		)
+		(property "MPN" "0402B104K160HI"
 			(at 146.05 116.84 0)
 			(effects
@@
 			)
 		)
+		(property "MPN" "RC0402JR-07100KL"
+			(at 128.27 132.08 0)
+			(effects
+				(font
+					(size 1.27 1.27)
+				)
+				(hide yes)
+			)
+		)
 		(pin "2"
 		)
@@
 			)
 		)
+		(property "MPN" "NCU15XH103F6SRC"
+			(at 128.27 124.46 0)
+			(effects
+				(font
+					(size 1.27 1.27)
+				)
+				(hide yes)
+			)
+		)
 		(pin "2"
 		)
@@
 			)
 		)
+		(property "MPN" "ADC081C021CIMM/NOPB"
+			(at 149.86 130.81 0)
+			(effects
+				(font
+					(size 1.27 1.27)
+				)
+				(hide yes)
+			)
+		)
 		(pin "2"
 		)
@@
 			(at 128.27 68.58 0)
 			(effects
+				(font
+					(size 1.27 1.27)
+				)
+				(hide yes)
+			)
+		)
+		(property "MPN" "0402B104K160HI"
+			(at 128.27 68.58 0)
+			(effects
