File: LoRa Module/LoRa Module.kicad_sch (KiCad schematic)
At the start: 8 parts, among them J1 Conn_MB

Commit message: Add part numbers to remaining PCBs, change part numbers on sensor board, redo strain adc layout
Parts:
- C1: MPN (none) -> CL05B104KP5NNNC
- C2: MPN (none) -> GRM155R60J475ME47D
- J1: MPN (none) -> B5B-XH-A
- R1, R2: MPN (none) -> RC0402JR-0710KL
Changed lines of the file:
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@@
+			)
+		)
+		(property "MPN" ""
+			(at 156.21 102.87 0)
+			(effects
+				(font
+					(size 1.27 1.27)
+				)
+				(hide yes)
 			)
 		)
@@
 			)
 		)
+		(property "MPN" "GRM155R60J475ME47D"
+			(at 142.24 93.98 0)
+			(effects
+				(font
+					(size 1.27 1.27)
+				)
+				(hide yes)
+			)
+		)
 		(pin "1"
 		)
@@
 		)
 		(property "Description" "Jumper, 2-pole, closed/bridged"
+			(at 180.34 100.33 0)
+			(effects
+				(font
+					(size 1.27 1.27)
+				)
+				(hide yes)
+			)
+		)
+		(property "MPN" ""
 			(at 180.34 100.33 0)
 			(effects
@@
 			)
 		)
+		(property "MPN" ""
+			(at 180.34 102.87 0)
+			(effects
+				(font
+					(size 1.27 1.27)
+				)
+				(hide yes)
+			)
+		)
 		(pin "2"
 		)
@@
 			)
 		)
+		(property "MPN" "B5B-XH-A"
+			(at 118.11 104.14 0)
+			(effects
+				(font
+					(size 1.27 1.27)
+				)
+				(hide yes)
+			)
+		)
 		(pin "1"
 		)
@@
 			)
 		)
+		(property "MPN" "RC0402JR-0710KL"
+			(at 173.99 96.52 0)
+			(effects
+				(font
+					(size 1.27 1.27)
+				)
+				(hide yes)
+			)
+		)
 		(pin "1"
 		)
@@
 			)
 		)
+		(property "MPN" "RC0402JR-0710KL"
+			(at 173.99 106.68 0)
+			(effects
+				(font
+					(size 1.27 1.27)
+				)
+				(hide yes)
+			)
+		)
 		(pin "1"
 		)
@@
 			(at 137.16 93.98 0)
 			(effects
+				(font
+					(size 1.27 1.27)
+				)
+				(hide yes)
+			)
+		)
+		(property "MPN" "CL05B104KP5NNNC"
+			(at 137.16 93.98 0)
+			(effects
