File: Motherboard/Motherboard.kicad_sch (KiCad schematic)
At the start: 30 parts, among them J1 Conn_RF, J2 Conn_Power, J3 Micro_SD_Card, J4 Conn_SW, J5 Conn_Strain, J6 Conn_Sensors, J7 Conn_Solar, J8 Conn_Cam, SW1 NRST, SW2 BOOT0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

Commit message: Add part numbers to remaining PCBs, change part numbers on sensor board, redo strain adc layout
Parts:
- C1, C11, C13, C14, C2, C3, C4: MPN (none) -> CL05B104KP5NNNC
- C12: MPN (none) -> GRM155R70J105KA12D
- C15: MPN (none) -> CL05A106MQ5NUNC
- C16, C18: MPN (none) -> GRM155R60J475ME47D
- C17: MPN (none) -> GRM1555C1H561JA01D
- J1, J5: MPN (none) -> B5B-XH-A
- J2: MPN (none) -> B2B-XH-A
- J3: MPN (none) -> MSD-1-A
- J4: MPN (none) -> 5-146274-4
- J6, J7: MPN (none) -> B4B-XH-A
- J8: MPN (none) -> B6B-XH-A
- L2: MPN (none) -> MCEE1005T1R0MHN
- R1: MPN (none) -> RC0402JR-0710KL
- R2, R3: MPN (none) -> RC0402JR-07560RL
- U1: MPN (none) -> STM32L431RCT6
- U2: MPN (none) -> MIC23050-SYML-TR
Changed lines of the file:
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@@
 			)
 		)
-		(property "MPN" ""
+		(property "MPN" "STM32L431RCT6"
 			(at 91.44 73.66 0)
 			(effects
@@
 			)
 		)
-		(property "MPN" ""
+		(property "MPN" "GRM155R60J475ME47D"
 			(at 237.49 78.74 0)
 			(effects
@@
 			)
 		)
-		(property "MPN" ""
+		(property "MPN" "CL05B104KP5NNNC"
 			(at 240.03 48.26 0)
 			(effects
@@
 			)
 		)
+		(property "MPN" "RC0402JR-07560RL"
+			(at 179.07 78.74 0)
+			(effects
+				(font
+					(size 1.27 1.27)
+				)
+				(hide yes)
+			)
+		)
 		(pin "1"
 		)
@@
 			)
 		)
-		(property "MPN" ""
+		(property "MPN" "GRM155R70J105KA12D"
 			(at 205.74 48.26 0)
 			(effects
@@
 			)
 		)
-		(property "MPN" ""
+		(property "MPN" "CL05B104KP5NNNC"
 			(at 219.71 48.26 0)
 			(effects
@@
 			)
 		)
-		(property "MPN" ""
+		(property "MPN" "MSD-1-A"
 			(at 223.52 128.27 0)
 			(effects
@@
 			)
 		)
-		(property "MPN" ""
+		(property "MPN" "GRM1555C1H561JA01D"
 			(at 204.47 81.28 0)
 			(effects
@@
 			)
 		)
+		(property "MPN" "RC0402JR-07560RL"
+			(at 123.19 83.82 90)
+			(effects
+				(font
+					(size 1.27 1.27)
+				)
+				(hide yes)
+			)
+		)
 		(pin "1"
 		)
@@
 			)
 		)
-		(property "MPN" ""
+		(property "MPN" "B5B-XH-A"
 			(at 64.77 149.86 0)
 			(effects
@@
 			)
 		)
-		(property "MPN" ""
+		(property "MPN" "B2B-XH-A"
 			(at 250.19 74.93 0)
 			(effects
@@
 			)
 		)
-		(property "MPN" ""
+		(property "MPN" "CL05B104KP5NNNC"
 			(at 250.19 48.26 0)
 			(effects
@@
 			)
 		)
-		(property "MPN" ""
+		(property "MPN" "MCEE1005T1R0MHN"
 			(at 205.74 74.93 90)
 			(effects
@@
 			)
 		)
-		(property "MPN" ""
+		(property "MPN" "RC0402JR-0710KL"
 			(at 60.96 46.99 0)
 			(effects
@@
 			)
 		)
-		(property "MPN" ""
+		(property "MPN" "CL05B104KP5NNNC"
 			(at 55.88 36.83 90)
 			(effects
@@
 			)
 		)
-		(property "MPN" ""
+		(property "MPN" "GRM155R60J475ME47D"
 			(at 194.31 78.74 0)
 			(effects
@@
 			)
 		)
-		(property "MPN" ""
+		(property "MPN" "B4B-XH-A"
 			(at 102.87 149.86 0)
 			(effects
@@
 			)
 		)
-		(property "MPN" ""
+		(property "MPN" "CL05A106MQ5NUNC"
 			(at 260.35 48.26 0)
 			(effects
@@
 			)
 		)
-		(property "MPN" ""
+		(property "MPN" "B5B-XH-A"
 			(at 64.77 171.45 0)
 			(effects
@@
 			)
 		)
-		(property "MPN" ""
+		(property "MPN" "MIC23050-SYML-TR"
 			(at 219.71 80.01 0)
 			(effects
@@
 			)
 		)
-		(property "MPN" ""
+		(property "MPN" "B4B-XH-A"
 			(at 102.87 172.72 0)
 			(effects
@@
 			)
 		)
-		(property "MPN" ""
+		(property "MPN" "CL05B104KP5NNNC"
 			(at 195.58 48.26 0)
 			(effects
@@
 			)
 		)
-		(property "MPN" ""
+		(property "MPN" "CL05B104KP5NNNC"
 			(at 180.34 48.26 0)
 			(effects
@@
 			)
 		)
-		(property "MPN" ""
+		(property "MPN" "B6B-XH-A"
 			(at 137.16 158.75 0)
 			(effects
@@
 			)
 		)
-		(property "MPN" ""
+		(property "MPN" "CL05B104KP5NNNC"
 			(at 229.87 48.26 0)
 			(effects
@@
 			)
 		)
-		(property "MPN" ""
+		(property "MPN" "5-146274-4"
 			(at 127 66.04 0)
 			(effects
