File: Ground RF/Ground RF Controller.kicad_pcb (KiCad board)
At the start: 2 copper layers, 0 parts

Commit message: v2.0.0 Ground RF finished
Parts:
- added C1: 100n, Capacitor_SMD:C_0402_1005Metric, F.Cu at (115.2, 114.7)
- added C2: 4.7uF, Capacitor_SMD:C_0402_1005Metric, F.Cu at (134.6, 99.8)
- added C20: 100n, Capacitor_SMD:C_0402_1005Metric, F.Cu at (134.6, 101.6)
- added C3: 100n, Capacitor_SMD:C_0402_1005Metric, F.Cu at (116.2, 114.7)
- added C4: 4.7uF, Capacitor_SMD:C_0402_1005Metric, F.Cu at (116.7, 112.6)
- added C6: 100n, Capacitor_SMD:C_0402_1005Metric, F.Cu at (115.7, 112.6)
- added C7: 4.7uF, Capacitor_SMD:C_0402_1005Metric, F.Cu at (117.4, 111.1)
- added C8: 100n, Capacitor_SMD:C_0402_1005Metric, F.Cu at (117.4, 110.1)
- added D2: LED, LED_SMD:LED_0603_1608Metric, F.Cu at (115.6, 108.0)
- added D3: LED, LED_SMD:LED_0603_1608Metric, F.Cu at (115.7, 106.4)
- added D6: SP0503BAHTG, Ground RF Controller:SOT143, F.Cu at (112.9, 113.7)
- added G***: LOGO, LOGO, F.Cu at (122.3, 117.5)
- added G***: LOGO, LOGO, F.Cu at (130.4, 115.6)
- added H3: MountingHole, MountingHole:MountingHole_2.7mm_M2.5, F.Cu at (136.0, 118.3)
- added H3: MountingHole, MountingHole:MountingHole_2.7mm_M2.5, F.Cu at (136.0, 84.7)
- added H3: MountingHole, MountingHole:MountingHole_2.7mm_M2.5, F.Cu at (104.0, 118.3)
- added H3: MountingHole, MountingHole:MountingHole_2.7mm_M2.5, F.Cu at (104.0, 84.7)
- added J3: USB_C_Receptacle_USB2.0_16P, Connector_USB:USB_C_Receptacle_GCT_USB4105-xx-A_16P_TopMnt_Horizontal, F.Cu at (106.0, 111.0)
- added JP1: Jumper_2_Bridged, Jumper:SolderJumper-2_P1.3mm_Open_RoundedPad1.0x1.5mm, F.Cu at (136.4, 89.5)
- added JP2: Jumper_2_Bridged, Jumper:SolderJumper-2_P1.3mm_Open_RoundedPad1.0x1.5mm, F.Cu at (136.4, 93.0)
- added R1: 5k1, Resistor_SMD:R_0603_1608Metric, F.Cu at (113.3, 109.6)
- added R10: 220, Resistor_SMD:R_1206_3216Metric, F.Cu at (127.0, 107.7)
- added R12: 5k1, Resistor_SMD:R_0603_1608Metric, F.Cu at (112.5, 107.2)
- added R2: 10k, Resistor_SMD:R_0402_1005Metric, F.Cu at (134.7, 88.5)
- added R3: 1k, Resistor_SMD:R_0805_2012Metric, F.Cu at (121.2, 114.0)
- added R4: 1k, Resistor_SMD:R_0805_2012Metric, F.Cu at (132.2, 109.6)
- added R5: 47.5k, Resistor_SMD:R_0402_1005Metric, F.Cu at (118.0, 114.4)
- added R6: 1k, Resistor_SMD:R_0805_2012Metric, F.Cu at (132.2, 106.8)
- added R7: 220, Resistor_SMD:R_1206_3216Metric, F.Cu at (127.0, 110.2)
- added R8: 10k, Resistor_SMD:R_0402_1005Metric, F.Cu at (134.7, 90.5)
- added R9: 22.1k, Resistor_SMD:R_0402_1005Metric, F.Cu at (119.2, 112.8)
- added U1: CP2102N-A02-GQFN28R, Package_DFN_QFN:QFN-28-1EP_5x5mm_P0.5mm_EP3.35x3.35mm, F.Cu at (121.5, 109.0)
- added U2: ~, Ground RF Controller:EBYTE-E220-900T22D, F.Cu at (118.0, 95.7)
Routing:
- net +5V: track 0.00 -> 22.5 mm
- net RXD: track 0.00 -> 19.6 mm
- net AUX: track 0.00 -> 17.3 mm, vias 0 -> 2
- net TXD: track 0.00 -> 15.6 mm
- net D+: track 0.00 -> 15.4 mm, vias 0 -> 2
- net D-: track 0.00 -> 14.5 mm
- net Net-(U1-TXD): track 0.00 -> 14.4 mm, vias 0 -> 2
- net Net-(U1-RXD): track 0.00 -> 13.4 mm, vias 0 -> 2
- net +3V3: track 0.00 -> 12.2 mm, vias 0 -> 5
- net Net-(D2-A): track 0.00 -> 12.0 mm, vias 0 -> 2
- net Net-(D3-A): track 0.00 -> 10.8 mm, vias 0 -> 2
- net Net-(JP2-A): track 0.00 -> 5.29 mm
- net Net-(J3-CC2): track 0.00 -> 4.81 mm, vias 0 -> 2
- net Net-(JP1-A): track 0.00 -> 4.62 mm
- net Net-(U1-VREGIN): track 0.00 -> 4.29 mm
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- added copper zone on In2.Cu, net +3V3
- added copper zone on B.Cu, net GND
- added copper zone on F.Cu, net GND
- added copper zone on In1.Cu, net GND
Other:
- board outline added: 36.1 x 37.8 mm
- copper layers 2 -> 4
- board text added: "ARYAN.ZAFER.2025"
- board text added: "Ground RF Controller v2.0.0"
