File: Ground RF/Ground RF Controller.kicad_pcb (KiCad board)
At the start: 4 copper layers, 36.1 x 37.8 mm, 33 parts, among them J3 USB_C_Receptacle_USB2.0_16P, U1 CP2102N-A02-GQFN28R

Commit message: PCB cleanup
Parts:
- moved D3 0.65 mm to (115.6, 105.8)
- moved D2 0.65 mm to (115.6, 107.3)
- moved R8 0.40 mm to (134.7, 90.8)
Routing:
- net Net-(D2-A): track 12.0 -> 12.7 mm
- net GND: vias 1 -> 3
Changed lines of the file:
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@@
 		(tags "resistor")
 		(property "Reference" "R3"
-			(at 0 -1.65 90)
+			(at -0.1 1.45 180)
 			(layer "F.SilkS")
 			(effects
@@
 	(footprint "Resistor_SMD:R_0402_1005Metric"
 		(layer "F.Cu")
-		(at 134.65 90.45 90)
+		(at 134.65 90.85 90)
 		(descr "Resistor SMD 0402 (1005 Metric), square (rectangular) end terminal, IPC-7351 nominal, (Body size source: IPC-SM-782 page 72, https://www.pcb-3d.com/wordpress/wp-content/uploads/ipc-sm-782a_amendment_1_and_2.pdf), generated with kicad-footprint-generator")
 		(tags "resistor")
@@
 	(footprint "LED_SMD:LED_0603_1608Metric"
 		(layer "F.Cu")
-		(at 115.65 106.4)
+		(at 115.6 105.75)
 		(descr "LED SMD 0603 (1608 Metric), square (rectangular) end terminal, IPC-7351 nominal, (Body size source: http://www.tortai-tech.com/upload/download/2011102023233369053.pdf), generated with kicad-footprint-generator")
 		(tags "LED")
 		(property "Reference" "D3"
-			(at 0 -1.43 0)
+			(at 1.9875 -0.55 0)
 			(layer "F.SilkS")
 			(effects
@@
 	(footprint "LED_SMD:LED_0603_1608Metric"
 		(layer "F.Cu")
-		(at 115.6375 108)
+		(at 115.5875 107.35)
 		(descr "LED SMD 0603 (1608 Metric), square (rectangular) end terminal, IPC-7351 nominal, (Body size source: http://www.tortai-tech.com/upload/download/2011102023233369053.pdf), generated with kicad-footprint-generator")
 		(tags "LED")
 		(property "Reference" "D2"
-			(at 0 -1.43 0)
+			(at 0.0125 1.15 0)
 			(layer "F.SilkS")
 			(effects
@@
 	)
 	(via
-		(at 113.05 115.6)
+		(at 137.2 91.25)
+		(size 0.6)
+		(drill 0.3)
+		(layers "F.Cu" "B.Cu")
+		(free yes)
+		(net 2)
+	)
+	(via
+		(at 133.6 91.95)
+		(size 0.6)
+		(drill 0.3)
+		(layers "F.Cu" "B.Cu")
+		(free yes)
+		(net 2)
+	)
+	(via
+		(at 113.1 114.2)
 		(size 0.6)
 		(drill 0.3)
@@
 	)
 	(segment
-		(start 116.425 108)
-		(end 117.6 108)
+		(start 116.375 107.35)
+		(end 117.05 107.35)
 		(width 0.2)
 		(layer "F.Cu")
@@
 	)
 	(segment
-		(start 117.6 108)
-		(end 117.7 108.1)
+		(start 117.05 107.35)
+		(end 117.55 106.85)
 		(width 0.2)
 		(layer "F.Cu")
@@
 	)
 	(via
-		(at 117.7 108.1)
+		(at 117.55 106.85)
 		(size 0.6)
 		(drill 0.3)
@@
 	)
 	(segment
-		(start 122.1 108.1)
+		(start 120.85 106.85)
 		(end 125.55 111.55)
 		(width 0.2)
@@
 	)
 	(segment
-		(start 117.7 108.1)
-		(end 122.1 108.1)
+		(start 117.55 106.85)
+		(end 120.85 106.85)
 		(width 0.2)
 		(layer "B.Cu")
@@
 	)
 	(segment
-		(start 117.55 106.4)
-		(end 117.85 106.7)
+		(start 116.4875 105.85)
+		(end 116.3875 105.75)
 		(width 0.2)
 		(layer "F.Cu")
@@
 	)
 	(segment
-		(start 116.4375 106.4)
-		(end 117.55 106.4)
+		(start 117.65 105.85)
+		(end 116.4875 105.85)
 		(width 0.2)
 		(layer "F.Cu")
@@
 	)
 	(via
-		(at 117.85 106.7)
+		(at 117.65 105.85)
 		(size 0.6)
 		(drill 0.3)
@@
 	)
 	(segment
-		(start 117.85 106.7)
-		(end 125.15 106.7)
+		(start 125.55 106.3)
+		(end 118.1 106.3)
 		(width 0.2)
 		(layer "B.Cu")
@@
 	)
 	(segment
-		(start 125.15 106.7)
-		(end 125.55 106.3)
+		(start 118.1 106.3)
+		(end 117.65 105.85)
 		(width 0.2)
 		(layer "B.Cu")
@@
 	)
 	(segment
-		(start 109.68 110.25)
-		(end 110.95 110.25)
-		(width 0.2)
-		(layer "F.Cu")
-		(net 8)
-	)
-	(segment
 		(start 119.089 109.489)
 		(end 119.1 109.5)
@@
 	)
 	(segment
-		(start 110.95 110.25)
-		(end 113.325 112.625)
-		(width 0.2)
-		(layer "F.Cu")
-		(net 8)
-	)
-	(segment
 		(start 108.804 110.517176)
 		(end 109.071176 110.25)
@@
 	)
 	(segment
-		(start 113.325 112.625)
-		(end 113.86 112.625)
+		(start 108.804 110.982824)
+		(end 108.804 110.517176)
 		(width 0.2)
 		(layer "F.Cu")
@@
 	)
 	(segment
-		(start 108.804 110.982824)
-		(end 108.804 110.517176)
+		(start 109.68 110.25)
+		(end 110.95 110.25)
 		(width 0.2)
 		(layer "F.Cu")
@@
 	)
 	(segment
+		(start 113.325 112.625)
+		(end 113.86 112.625)
+		(width 0.2)
+		(layer "F.Cu")
+		(net 8)
+	)
+	(segment
+		(start 110.95 110.25)
+		(end 113.325 112.625)
+		(width 0.2)
+		(layer "F.Cu")
+		(net 8)
+	)
+	(segment
 		(start 109.071176 111.25)
 		(end 108.804 110.982824)
@@
 	)
 	(segment
-		(start 132.5 89.92)
-		(end 134.63 89.92)
+		(start 135.85 91.14)
+		(end 135.05 90.34)
+		(width 0.2)
+		(layer "F.Cu")
+		(net 14)
+	)
+	(segment
+		(start 132.79 90.34)
+		(end 132.5 90.63)
 		(width 0.2)
 		(layer "F.Cu")
@@
 	)
 	(segment
-		(start 134.63 89.92)
-		(end 134.65 89.94)
+		(start 134.65 90.34)
+		(end 132.79 90.34)
 		(width 0.2)
 		(layer "F.Cu")
@@
 	)
 	(segment
-		(start 134.65 89.94)
-		(end 135.85 91.14)
+		(start 135.05 90.34)
+		(end 134.65 90.34)
 		(width 0.2)
 		(layer "F.Cu")
@@
 		(hatch edge 0.5)
 		(connect_pads
-			(clearance 0.1)
+			(clearance 0.25)
 		)
-		(min_thickness 0.1)
+		(min_thickness 0.25)
 		(filled_areas_thickness no)
 		(fill yes
-			(thermal_gap 0.1)
-			(thermal_bridge_width 0.1)
+			(thermal_gap 0.5)
+			(thermal_bridge_width 0.5)
 		)
 		(polygon
@@
 		(priority 3)
 		(connect_pads
-			(clearance 0.1)
+			(clearance 0.25)
 		)
-		(min_thickness 0.1)
+		(min_thickness 0.25)
 		(filled_areas_thickness no)
 		(fill yes
-			(thermal_gap 0.1)
-			(thermal_bridge_width 0.1)
+			(thermal_gap 0.5)
+			(thermal_bridge_width 0.5)
 		)
 		(polygon
@@
 		(priority 1)
 		(connect_pads
-			(clearance 0.1)
+			(clearance 0.25)
 		)
-		(min_thickness 0.1)
+		(min_thickness 0.25)
 		(filled_areas_thickness no)
 		(fill yes
-			(thermal_gap 0.1)
-			(thermal_bridge_width 0.1)
+			(thermal_gap 0.5)
+			(thermal_bridge_width 0.5)
 		)
 		(polygon
@@
 		(priority 2)
 		(connect_pads
-			(clearance 0.1)
+			(clearance 0.25)
 		)
-		(min_thickness 0.1)
+		(min_thickness 0.25)
 		(filled_areas_thickness no)
 		(fill yes
-			(thermal_gap 0.1)
-			(thermal_bridge_width 0.1)
+			(thermal_gap 0.5)
+			(thermal_bridge_width 0.5)
 		)
 		(polygon
